File: KiCad/ozone12864.kicad_sch (KiCad schematic)
At the start: 57 parts, among them J1 DCJACK, J10 TWELITE_VCC_JUMPER, J11 Conn_01x13_Female, J12 Screw_Terminal_01x02, J13 SD_CARD_MODULE, J2 DEBUG, J3 Conn_01x08_Female, J4 MODE_JUMPER, J5 USBSERIAL, J6 ANALOG_SELECT, J7 Conn_01x13_Female, J8 Conn_01x13_Male, J9 Conn_01x13_Male, Q1 Q_NMOS_GSD, Q3 Si4542DY, SW1 SW_SPDT, SW2 SW_DPST, SW3 A, SW4 B, SW5 OK, U1 ESP-WROOM-32, U2 JLX12864G-LCD, U3 TWELITE_DIP_APP_TWELITE_PINNA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, U5 NJM2845DL1-33, U6 DCDC Up/Down

Commit message: update schematic
Parts:
- added D2: D_Schottky, Diode_SMD:D_SOD-123, symbol Device:D_Schottky
- added R4, R5: 510k, Resistor_SMD:R_0603_1608Metric, symbol Device:R
- renumbered D2 to D3, R3 to R1, R4 to R15, R8 to R16, R27 to R17, R1 to R2, R2 to R3, R5 to R7, R7 to R8
Connections:
- net GND: now also R4.1
- net VIN: no longer C8.1, D1.1 (K), J11.10 (Pin_10), R16.2, U6.1 (VIN), U6.3 (EN)
- net at U1.23 (IO15): now also R16.2
- net at Q3.3 (1), R14.2, SW1.2 (B)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: no longer J11.7 (Pin_7), U1.6 (IO34)
- new net: R4.2, R5.2, U1.6 (IO34)
- new net: D2.2 (A), J11.10 (Pin_10), R5.1
- new net: D1.1 (K), D2.1 (K), U6.1 (VIN), U6.3 (EN)
Other:
- note added: "VIN MONITOR"
- note removed: "BACKUP BATTERY MONITOR"
- moved on the sheet: BT1, BZ1, C1, C10, C11, C12, C2, C3, C4, C5, C6, C7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

Commit message: fix pcb bug / add arduino sketch
Connections:
- net VIN: now also C8.1, D1.1 (K), D2.1 (K), U6.1 (VIN), U6.3 (EN)
Changed lines of the file:
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@@
   (junction (at 106.172 139.446) (diameter 0) (color 0 0 0 0)
+  )
+  (junction (at 192.532 205.994) (diameter 0) (color 0 0 0 0)
   )
   (junction (at 88.392 161.036) (diameter 0) (color 0 0 0 0)
@@
     (stroke (width 0) (type default))
   )
-  (wire (pts (xy 192.405 207.264) (xy 192.405 205.994))
-    (stroke (width 0) (type default))
-  )
   (wire (pts (xy 262.382 94.996) (xy 320.802 94.996))
     (stroke (width 0) (type default))
@@
     (stroke (width 0) (type default))
   )
+  (wire (pts (xy 192.532 205.994) (xy 192.532 207.264))
+    (stroke (width 0) (type default))
+  )
   (wire (pts (xy 271.272 131.826) (xy 271.272 130.556))
     (stroke (width 0) (type default))
@@
     (stroke (width 0) (type default))
   )
-  (wire (pts (xy 182.88 205.994) (xy 201.93 205.994))
+  (wire (pts (xy 182.88 205.994) (xy 192.532 205.994))
     (stroke (width 0) (type default))
   )
@@
   )
   (wire (pts (xy 104.902 169.926) (xy 104.902 134.366))
+    (stroke (width 0) (type default))
+  )
+  (wire (pts (xy 192.532 205.994) (xy 201.93 205.994))
     (stroke (width 0) (type default))
   )
@@
     (property "Intersheetrefs" "${INTERSHEET_REFS}" (at 145.542 141.986 0)
       (effects (font (size 1.27 1.27)) hide)
+    )
+  )
+  (global_label "VIN" (shape input) (at 182.88 198.374 0) (fields_autoplaced)
+    (effects (font (size 2.0066 2.0066)) (justify left))
+    (property "Intersheetrefs" "${INTERSHEET_REFS}" (at 191.34 198.374 0)
+      (effects (font (size 1.27 1.27)) (justify left) hide)
     )
   )
@@
     )
   )
-  (symbol (lib_id "ozone12864-rescue:CP-Device") (at 192.405 211.074 0) (unit 1)
-    (in_bom yes) (on_board yes) (dnp no)
-    (property "Reference" "C8" (at 195.4022 209.9056 0)
+  (symbol (lib_id "ozone12864-rescue:CP-Device") (at 192.532 211.074 0) (unit 1)
+    (in_bom yes) (on_board yes) (dnp no)
+    (property "Reference" "C8" (at 195.5292 209.9056 0)
       (effects (font (size 1.27 1.27)) (justify left))
     )
-    (property "Value" "220uF" (at 195.4022 212.217 0)
+    (property "Value" "220uF" (at 195.5292 212.217 0)
       (effects (font (size 1.27 1.27)) (justify left))
     )
-    (property "Footprint" "Capacitor_THT:CP_Radial_D5.0mm_P2.00mm" (at 193.3702 214.884 0)
-      (effects (font (size 1.27 1.27)) hide)
-    )
-    (property "Datasheet" "~" (at 192.405 211.074 0)
+    (property "Footprint" "Capacitor_THT:CP_Radial_D5.0mm_P2.00mm" (at 193.4972 214.884 0)
+      (effects (font (size 1.27 1.27)) hide)
+    )
+    (property "Datasheet" "~" (at 192.532 211.074 0)
       (effects (font (size 1.27 1.27)) hide)
     )
@@
     )
   )
-  (symbol (lib_id "power:GND") (at 192.405 214.884 0) (unit 1)
-    (in_bom yes) (on_board yes) (dnp no)
-    (property "Reference" "#PWR0131" (at 192.405 221.234 0)
-      (effects (font (size 1.27 1.27)) hide)
-    )
-    (property "Value" "GND" (at 192.532 219.2782 0)
-      (effects (font (size 1.27 1.27)))
-    )
-    (property "Footprint" "" (at 192.405 214.884 0)
-      (effects (font (size 1.27 1.27)) hide)
-    )
-    (property "Datasheet" "" (at 192.405 214.884 0)
-      (effects (font (size 1.27 1.27)) hide)
-    )
+  (symbol (lib_id "power:GND") (at 192.532 214.884 0) (unit 1)
+    (in_bom yes) (on_board yes) (dnp no)
+    (property "Reference" "#PWR0131" (at 192.532 221.234 0)
+      (effects (font (size 1.27 1.27)) hide)
+    )
+    (property "Value" "GND" (at 192.659 219.2782 0)
+      (effects (font (size 1.27 1.27)))
+    )
+    (property "Footprint" "" (at 192.532 214.884 0)
+      (effects (font (size 1.27 1.27)) hide)
+    )
+    (property "Datasheet" "" (at 192.532 214.884 0)
+      (effects (font (size 1.27 1.27)) hide)
+    )
