File: KiCad/ozone12864.kicad_pcb (KiCad board)
At the start: 2 copper layers, 70.1 x 138 mm, 66 parts, among them J1 DCJACK, J11 Conn_01x13_Female, J12 Screw_Terminal_01x02, J13 SD_CARD_MODULE, J2 DEBUG, J3 Conn_01x08_Female, J5 USBSERIAL, J7 Conn_01x13_Female, J9 Conn_01x13_Male, Q1 Q_NMOS_GSD, SW1 SW_SPDT, SW2 SW_DPST, SW3 A, SW4 B, SW5 OK, U1 ESP-WROOM-32, U2 JLX12864G-LCD, U4 DC-DC BOOSTUP, U5 NJM2845DL1-33

Commit message: update to ver.202307 version
Parts:
- removed the BZ1 at (121.6, 129.2)
- removed JP1: Jumper_NC_Small, Jumper:SolderJumper-2_P1.3mm_Bridged_RoundedPad1.0x1.5mm
- removed SW1: SW_SPDT, library:SS-12F23_SLIDE_SWITCH
- removed U4: DC-DC BOOSTUP, Connector_PinHeader_2.54mm:PinHeader_1x03_P2.54mm_Vertical
- added Q3: Si4542DY, Package_SO:SO-8_5.3x6.2mm_P1.27mm, F.Cu at (127.9, 129.0)
- added R10: 1k, Resistor_SMD:R_0603_1608Metric, F.Cu at (133.0, 126.7)
- added R11: 1k, Resistor_SMD:R_0603_1608Metric, F.Cu at (133.0, 131.2)
- added R12: 10k, Resistor_SMD:R_0603_1608Metric, F.Cu at (132.2, 122.5)
- added R13: 1k, Resistor_SMD:R_0603_1608Metric, F.Cu at (133.0, 135.3)
- added R14: 10k, Resistor_SMD:R_0603_1608Metric, F.Cu at (122.7, 122.5)
- added REF**: MountingHole_2.7mm_M2.5_ISO14580_Pad, MountingHole:MountingHole_2.7mm_M2.5_ISO14580_Pad, F.Cu at (86.5, 177.0)
- added U6: DCDC Up/Down, library:TPS63020_Module_Both_Strawberrylinux_Taobao, F.Cu at (103.9, 121.3)
- moved R8 82.0 mm to (83.7, 106.5)
- moved C12 59.4 mm to (79.0, 118.5), turned to 180 degrees
- moved C8 57.1 mm to (85.5, 118.5), turned to 180 degrees
- moved BZ1 39.0 mm to (82.6, 128.5)
- moved D1 33.3 mm to (89.3, 106.5), turned to 0 degrees
- moved J5 1.00 mm to (76.5, 139.8)
Connections:
- net CONTROL renamed RELAYCONTROL
- C8 pad 1: Net-(J11-Pin_5) -> VIN
- D1 pad 1: Net-(D1-K) -> VIN
- D1 pad 2: VIN -> Net-(D1-A)
- J11 pad 5: Net-(J11-Pin_5) -> Net-(D1-A)
- J11 pad 8: Net-(D1-K) -> +3V3
- R5 pad 1: Net-(J11-Pin_5) -> Net-(D1-A)
- SW2 pad 1: Net-(D1-K) -> Net-(J11-Pin_7)
- SW2 pad 2: +3V3 -> OFF SW DETECT
- SW2 pad 3: Net-(D1-K) -> Net-(J11-Pin_7)
- U1 pad 10: unconnected-(U1-IO25-Pad10) -> OFF SW DETECT
- U1 pad 26: unconnected-(U1-IO4-Pad26) -> _POWERDOWN
Routing:
- net Net-(J11-Pin_5): track 129.2 -> 0.00 mm, vias 2 -> 0
- net VIN: track 225.0 -> 96.6 mm, vias 13 -> 3
- net OFF SW DETECT: track 0.00 -> 119.9 mm, vias 0 -> 3
- net Net-(D1-A): track 0.00 -> 106.8 mm, vias 0 -> 4
- net Net-(D1-K): track 96.2 -> 0.00 mm, vias 2 -> 0
- net _POWERDOWN: track 0.00 -> 89.4 mm, vias 0 -> 5
- net Net-(J11-Pin_7): track 122.1 -> 200.5 mm, vias 4 -> 6
- net Net-(U2-LEDA): track 108.5 -> 38.6 mm, vias 3 -> 1
- net Net-(Q3A-D-Pad7): track 0.00 -> 30.0 mm
- net Net-(Q3B-G): track 0.00 -> 14.1 mm
- net RELAYCONTROL: track 101.2 -> 112.7 mm
- net +3V3: track 304.5 -> 314.2 mm, vias 5 -> 6
- net GND: track 223.3 -> 232.3 mm, vias 8 -> 9
- net Net-(Q3A-G): track 0.00 -> 7.20 mm
- net Net-(J2-Pin_7): track 96.9 -> 102.8 mm
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Other:
- outline, holes or cut-outs redrawn
- board text added: "10k x 2"
- board text added: "1k x 3"
- board text added: "510k x 4"
- board text added: "GND 3.3 KEY VIN"
- board text added: "VBackup"
- board text added: "Vgas Vref Temp SDA VBATT"
- board text removed: "SDA SCL GND BAT 3VIN VIN"
- board text removed: "VI GND VO"

Commit message: fix pcb bug / add arduino sketch
Parts:
- added D2: D_Schottky, Diode_SMD:D_SOD-123, F.Cu at (75.3, 112.8)
- added OSHW: 1.1, library:OSHW_LOGL_SYLK_5mm, F.Cu at (100.0, 207.6)
- added R4: 510k, Resistor_SMD:R_0603_1608Metric, F.Cu at (111.0, 164.9)
- added R5: 510k, Resistor_SMD:R_0603_1608Metric, F.Cu at (111.0, 167.4)
- moved D1 19.1 mm to (71.4, 113.0), turned to 90 degrees
- moved R17 0.53 mm to (107.8, 153.5)
- turned C12 to 90 degrees
- turned C8 to 90 degrees
- renumbered D2 to D3, R3 to R1, R4 to R15, R8 to R16, R27 to R17, R1 to R2, R2 to R3, R5 to R7, R7 to R8
Connections:
- J11 pad 10: VIN -> Net-(D2-A)
- J11 pad 7: Net-(J11-Pin_7) -> unconnected-(J11-Pin_7-Pad7)
- Q3 pad 3: Net-(J11-Pin_7) -> Net-(Q3B-1)
- R14 pad 2: Net-(J11-Pin_7) -> Net-(Q3B-1)
- R16 pad 2: VIN -> Net-(U1-IO15)
- SW2 pad 1: Net-(J11-Pin_7) -> Net-(Q3B-1)
- SW2 pad 3: Net-(J11-Pin_7) -> Net-(Q3B-1)
- U1 pad 23: unconnected-(U1-IO15-Pad23) -> Net-(U1-IO15)
- U1 pad 6: Net-(J11-Pin_7) -> Net-(U1-IO34)
- U6 pad 5: Net-(J11-Pin_7) -> Net-(Q3B-1)
Routing:
- net Net-(J11-Pin_7): track 200.5 -> 0.00 mm, vias 6 -> 0
- net Net-(D2-A): track 0.00 -> 112.7 mm, vias 0 -> 2
- net Net-(U1-IO15): track 0.00 -> 91.2 mm, vias 0 -> 2
- net Net-(U1-IO34): track 0.00 -> 58.0 mm, vias 0 -> 4
- net Net-(Q3B-1): track 0.00 -> 50.4 mm, vias 0 -> 1
- net Net-(D1-A): track 106.8 -> 130.0 mm
- net VIN: track 96.6 -> 116.1 mm, vias 3 -> 4
- net +3V3: track 314.2 -> 323.4 mm, vias 6 -> 7
- net GND: track 232.3 -> 239.3 mm, vias 9 -> 10
- net Net-(J13-Pin_3): track 143.5 -> 140.4 mm
- net Net-(U1-IO13): track 46.2 -> 48.9 mm
- net Net-(U1-IO17): track 88.4 -> 86.0 mm
- net TX: track 131.5 -> 133.6 mm
- net RELAYCONTROL: track 112.7 -> 110.7 mm
- net Net-(U1-IO2): track 39.5 -> 41.5 mm
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Other:
- board text added: "GND 3.3 KEY VIN CTL RX TX"
- board text added: "NOT CUT"
- board text added: "ozone12864 Ver.20230822"
- board text removed: "GND 3.3 KEY VIN"

Commit message: PCB pattern bug fix
Routing:
- net Net-(D2-A): track 112.7 -> 114.1 mm
- net VIN: track 116.1 -> 117.1 mm
Other:
- board text added: "ozone12864 Ver.20230926"
- board text removed: "ozone12864 Ver.20230822"

Commit message: LovyanGFX test
Parts:
- J11: moved to B.Cu
- turned J11 to 90 degrees
Other:
- board size 70.1 x 138 mm -> 72.8 x 138 mm
- board text added: "VCUT LINE"
- board text removed: "NOT CUT"
